File: HackPad.kicad_sch (KiCad schematic)
At the start: 11 parts, among them U1 MOUDLE-SEEEDUINO-XIAO

Commit message: Added switches
Parts:
- D1, D2, D3, D4: footprint (none) -> Diode_SMD:D_SOD-123
- F1: footprint (none) -> Capacitor_SMD:C_0805_2012Metric
- MX1, MX2, MX3, MX4: footprint (none) -> MX_Alps_Hybrid:MX-10U-NoLED
- U1: footprint (none) -> random-keyboard-parts:Molex-0548190589
- USB1: footprint (none) -> XIAO_PCB:MOUDLE14P-2.54-21X17.8MM
Connections:
- net GND: now also USB1.1 (GND)
- net COL1: now reaches MX3.1 (COL)
- net COL1: now also MX2.1 (COL)
- net ROW0: now reaches D3.1 (K)
- net ROW0: now also D4.1 (K)
- net D+: now reaches USB1.3 (D+)
- net D-: now reaches USB1.4 (D-)
- net ROW1: now reaches D1.1 (K)
- net ROW1: now also D2.1 (K)
- net COL0: now reaches MX1.1 (COL)
- net COL0: now also MX4.1 (COL)
